Commit message: 更新模型

File: biped.urdf (robot description, URDF)
Before this commit: robot biped, 7 links, 6 joints
Links:
- link left_foot: mass 0.2 -> 0.08; geometry collision box size=0.1 0.06 0.04; visual box size=0.1 0.06 0.04
- link left_shin: mass 0.3 -> 0.10
- link left_thigh: mass 0.5 -> 0.12
- link right_foot: mass 0.2 -> 0.08; geometry collision box size=0.1 0.06 0.04; visual box size=0.1 0.06 0.04
- link right_shin: mass 0.3 -> 0.10
- link right_thigh: mass 0.5 -> 0.12
- link torso: mass 2.0 -> 0.25
Joints:
- joint left_hip: axis 1 0 0 -> 0 1 0; limit lower=-1.0 upper=1.0 effort=20 velocity=2.0 -> lower=-1.57 upper=1.57 effort=1.0 velocity=10.0
- joint left_knee: axis 1 0 0 -> 0 1 0; limit lower=0 upper=2.0 effort=15 velocity=2.0 -> lower=0 upper=1.57 effort=1.0 velocity=10.0
- joint right_hip: axis 1 0 0 -> 0 1 0; limit lower=-1.0 upper=1.0 effort=20 velocity=2.0 -> lower=-1.57 upper=1.57 effort=1.0 velocity=10.0
- joint right_knee: axis 1 0 0 -> 0 1 0; limit lower=0 upper=2.0 effort=15 velocity=2.0 -> lower=0 upper=1.57 effort=1.0 velocity=10.0
