Commit message: Rebuild biped training pipeline for ten SG90 servos

File: biped.urdf (robot description, URDF)
Before this commit: robot biped, 7 links, 6 joints
Links:
- added link left_ankle, mass 0.01; collision box size=0.022 0.018 0.018; visual box size=0.022 0.018 0.018
- added link left_hip, mass 0.012; collision box size=0.023 0.014 0.018; visual box size=0.023 0.014 0.018
- added link right_ankle, mass 0.01; collision box size=0.022 0.018 0.018; visual box size=0.022 0.018 0.018
- added link right_hip, mass 0.012; collision box size=0.023 0.014 0.018; visual box size=0.023 0.014 0.018
- link left_foot: mass 0.08 -> 0.015; geometry collision box size=0.06 0.04 0.006; visual box size=0.06 0.04 0.006
- link left_shin: mass 0.10 -> 0.018; geometry collision box size=0.014 0.018 0.055; visual box size=0.014 0.018 0.055
- link left_thigh: mass 0.12 -> 0.02; geometry collision box size=0.016 0.022 0.055; visual box size=0.016 0.022 0.055
- link right_foot: mass 0.08 -> 0.015; geometry collision box size=0.06 0.04 0.006; visual box size=0.06 0.04 0.006
- link right_shin: mass 0.10 -> 0.018; geometry collision box size=0.014 0.018 0.055; visual box size=0.014 0.018 0.055
- link right_thigh: mass 0.12 -> 0.02; geometry collision box size=0.016 0.022 0.055; visual box size=0.016 0.022 0.055
- link torso: mass 0.25 -> 0.1; geometry collision box size=0.045 0.07 0.055; visual box size=0.045 0.07 0.055
Joints:
- removed joint left_ankle
- removed joint left_hip
- removed joint right_ankle
- removed joint right_hip
- added joint left_ankle_pitch: type revolute, parent left_shin, child left_ankle, origin xyz=0 0 -0.055, axis 0 1 0, limit lower=-0.95 upper=0.65 effort=0.08 velocity=6.0
- added joint left_ankle_roll: type revolute, parent left_ankle, child left_foot, origin xyz=0 0 0, axis 1 0 0, limit lower=-0.45 upper=0.45 effort=0.08 velocity=6.0
- added joint left_hip_pitch: type revolute, parent left_hip, child left_thigh, origin xyz=0 0 -0.009, axis 0 1 0, limit lower=-0.85 upper=0.65 effort=0.08 velocity=6.0
- added joint left_hip_roll: type revolute, parent torso, child left_hip, origin xyz=0 0.03 -0.0275, axis 1 0 0, limit lower=-0.45 upper=0.45 effort=0.08 velocity=6.0
- added joint right_ankle_pitch: type revolute, parent right_shin, child right_ankle, origin xyz=0 0 -0.055, axis 0 1 0, limit lower=-0.95 upper=0.65 effort=0.08 velocity=6.0
- added joint right_ankle_roll: type revolute, parent right_ankle, child right_foot, origin xyz=0 0 0, axis 1 0 0, limit lower=-0.45 upper=0.45 effort=0.08 velocity=6.0
- added joint right_hip_pitch: type revolute, parent right_hip, child right_thigh, origin xyz=0 0 -0.009, axis 0 1 0, limit lower=-0.85 upper=0.65 effort=0.08 velocity=6.0
- added joint right_hip_roll: type revolute, parent torso, child right_hip, origin xyz=0 -0.03 -0.0275, axis 1 0 0, limit lower=-0.45 upper=0.45 effort=0.08 velocity=6.0
- joint left_knee: limit lower=0 upper=1.57 effort=1.0 velocity=10.0 -> lower=0.02 upper=1.5 effort=0.08 velocity=6.0; origin xyz=0 0 -0.15 rpy=0 0 0 -> xyz=0 0 -0.055
- joint right_knee: limit lower=0 upper=1.57 effort=1.0 velocity=10.0 -> lower=0.02 upper=1.5 effort=0.08 velocity=6.0; origin xyz=0 0 -0.15 rpy=0 0 0 -> xyz=0 0 -0.055
